File: TasmotaGlow/TasmotaGlow.kicad_pcb (KiCad board)
At the start: 2 copper layers, 48.8 x 41.8 mm, 13 parts, among them J1 Conn_01x04, J2 Conn_01x04, J3 ResetPinout, Q1 BUZ11, Q2 BUZ11, U1 ESP-01v090, U2 LD1117S33TR_SOT223

Commit message: updated circuit
Parts:
- removed the G*** at (98.2, 120.9)
- added PS1: IRM-10-12, Converter_ACDC:Converter_ACDC_MeanWell_IRM-10-xx_THT, F.Cu at (125.7, 110.6)
- G***: moved to F.Cu
- J1: value Conn_01x04 -> Conn_01x02; footprint Connector_Phoenix_MC_HighVoltage:PhoenixContact_MCV_1,5_4-G-5.08_1x04_P5.08mm_Vertical -> Connector_Phoenix_MC_HighVoltage:PhoenixContact_MCV_1,5_2-G-5.08_1x02_P5.08mm_Vertical
- moved C1 51.5 mm to (157.3, 68.0)
- moved J2 49.2 mm to (160.9, 112.0)
- moved U2 48.1 mm to (137.0, 63.3), turned to 180 degrees
- moved C2 43.5 mm to (145.9, 68.0), turned to 90 degrees
- moved G*** 41.1 mm to (163.2, 92.5), turned to 0 degrees
- moved R2 37.8 mm to (154.1, 82.4), turned to 90 degrees
- moved J3 37.6 mm to (108.2, 79.5)
- moved U1 33.8 mm to (163.2, 71.4)
- moved R1 28.2 mm to (146.1, 82.3), turned to 90 degrees
- moved Q2 18.4 mm to (146.1, 92.4)
- moved Q1 16.9 mm to (146.2, 105.3)
- moved J1 6.26 mm to (108.1, 101.1)
Connections:
- C2 pad 1: Net-(C2-Pad1) -> Net-(U1-VCC)
- J1 pad 1: /GND -> Net-(J1-Pin_1)
- J1 pad 2: /VCC -> Net-(J1-Pin_2)
- J2 pad 1: Net-(J2-Pad1) -> /VCC
- J2 pad 2: Net-(J2-Pad2) -> Net-(J2-Pin_2)
- J2 pad 3: Net-(J2-Pad3) -> /VCC
- Q1 pad 2: Net-(J2-Pad3) -> Net-(J2-Pin_2)
- R1 pad 2: Net-(C2-Pad1) -> Net-(U1-VCC)
- R2 pad 2: Net-(C2-Pad1) -> Net-(U1-VCC)
- U1 pad 1: Net-(J2-Pad1) -> unconnected-(U1-UTXD-Pad1)
- U1 pad 7: Net-(C2-Pad1) -> Net-(U1-VCC)
- U1 pad 8: Net-(J2-Pad2) -> unconnected-(U1-URXD-Pad8)
- U2 pad 2: Net-(C2-Pad1) -> Net-(U1-VCC)
Routing:
- net /VCC: track 16.5 -> 114.5 mm
- net Net-(C2-Pad1): track 43.9 -> 0.00 mm
- net Net-(J2-Pad1): track 38.7 -> 0.00 mm
- net Net-(U1-VCC): track 0.00 -> 37.6 mm
- net Net-(J1-Pin_2): track 0.00 -> 34.4 mm
- net Net-(J2-Pad2): track 30.6 -> 0.00 mm
- net Net-(J2-Pin_2): track 0.00 -> 29.6 mm
- net Net-(J2-Pin_4): track 15.0 -> 39.2 mm
- net Net-(J1-Pin_1): track 0.00 -> 21.5 mm
- net Net-(Q1-G): track 21.1 -> 42.3 mm
- net Net-(Q2-G): track 15.6 -> 33.2 mm
- net /GND: track 87.3 -> 103.8 mm
- net Net-(J3-Pin_1): track 43.4 -> 59.9 mm
- net Net-(J2-Pad3): track 14.2 -> 0.00 mm
- net Net-(U1-CH_PD): track 15.7 -> 20.5 mm
Other:
- board size 48.8 x 41.8 mm -> 91.3 x 58.7 mm
- net class Default removed
- board text added: "+"
- board text added: "-"
- board text added: "L"
- board text added: "N"
- board text added: "TasmotaGlow © 2025"
- board text removed: "(+)"
- board text removed: "(-)"
- board text removed: "3.3V"
- board text removed: "GND"
- board text removed: "Out"
- board text removed: "R"
- board text removed: "T"
