File: TasmotaGlow/TasmotaGlow.kicad_sch (KiCad schematic)
At the start: 11 parts, among them J1 Conn_01x04, J2 Conn_01x04, J3 ResetPinout, Q1 BUZ11, Q2 BUZ11, U1 ESP-01v090, U2 LD1117S33TR_SOT223

Commit message: updated circuit
Parts:
- removed J1: Conn_01x04, Connector_Phoenix_MC_HighVoltage:PhoenixContact_MCV_1,5_4-G-5.08_1x04_P5.08mm_Vertical, symbol Connector_Generic:Conn_01x04
- added J1: Conn_01x02, Connector_Phoenix_MC_HighVoltage:PhoenixContact_MCV_1,5_2-G-5.08_1x02_P5.08mm_Vertical, symbol Connector_Generic:Conn_01x02
- added PS1: IRM-10-12, Converter_ACDC:Converter_ACDC_MeanWell_IRM-10-xx_THT, symbol Converter_ACDC:IRM-10-12
Connections:
- net GND: now also PS1.3 (-Vo)
- net VCC: now also J2.1 (Pin_1), J2.3 (Pin_3), PS1.4 (+Vo)
- net at U1.1 (UTXD): no longer J2.1 (Pin_1)
- net at U1.8 (URXD): no longer J2.2 (Pin_2)
- net at Q1.2 (D): now also J2.2 (Pin_2); no longer J2.3 (Pin_3)
- new net: J1.1 (Pin_1), PS1.1 (AC/N)
- new net: J1.2 (Pin_2), PS1.2 (AC/L)
Other:
- title: TasmotaGeneric -> TasmotaGlow
